File: pcb/Stepper_motor.kicad_sch (KiCad schematic)
At the start: 27 parts

Commit message: Schema: connect MCU to buttons and stepper motor
Parts:
- added R32, R33: 10k, Resistor_SMD:R_0603_1608Metric, symbol Device:R
- added TP5: VREF, TCY_connectors:TestPoint_Pad_D0.5mm, symbol Connector:TestPoint
- C22, C25, C26: renamed from C?; footprint (none) -> Capacitor_SMD:C_0603_1608Metric
- C23: renamed from C?; footprint (none) -> Capacitor_SMD:C_0805_2012Metric
- C24: renamed from C?; footprint (none) -> Capacitor_SMD:CP_Elec_8x10
- D2: renamed from D?; value D_Schottky -> SKL110; footprint (none) -> Diode_SMD:D_SOD-123F
- L1: renamed from L?; footprint (none) -> TCY_passives:Laird_2520
- M1: renamed from M?; footprint (none) -> Connector_JST:JST_PH_S4B-PH-K_1x04_P2.00mm_Horizontal
- R23, R24, R25, R26, R27, R28, R29, R30, R31, R34: renamed from R?; footprint (none) -> Resistor_SMD:R_0603_1608Metric
- R35, R36: renamed from R?; footprint (none) -> Resistor_SMD:R_1206_3216Metric
- RV1: renamed from RV?; footprint (none) -> Potentiometer_SMD:Potentiometer_Bourns_3214J_Horizontal
- TP3, TP4, TP6, TP7: renamed from TP?; footprint (none) -> TCY_connectors:TestPoint_Pad_D0.5mm
- gave numbers to parts that had none: 2
Connections:
- net +12V: now also C24.1, C26.1
- net +3V3: no longer U9.18 (DECAY)
- net DIR: now also R32.1
- net GND: now also U9.18 (DECAY), R32.2, R33.2
- net REF: now also TP5.1
- net STEP: now also R33.1
- net VBUS: no longer C24.1, C26.1
Other:
- note added: "Motor is modified to bipolar. Due to this needs higher voltage for driving."
- note added: "Motor reference voltage is generated by STM32 DAC."
- note added: "Output of step-up shout be some where around 10-12V. It depends on stepper motor heat dissipation."
- note added: "Select microstepping by populating one of two rezistors for overy MODE input of stepper motor driver."
- note removed: "Motor is modified to bipolar Due to this needs higher voltage for driving"
- note removed: "select microstepping by populating one of two rezistors for overy MODE input of stepper motor driver"
- company: (none) -> Author: Petr Malaník
- title: (none) -> Hepheatus - Solder paste dispensor
- moved on the sheet: C25, R25, R26, R27, R28, R29, R30, R31, R35, R36, TP4

Commit message: PCB: Basic routing done
Parts:
- added C27: 100nF, Capacitor_SMD:C_0603_1608Metric, symbol Device:C
- added C28: 100uF/16V, Capacitor_Tantalum_SMD:CP_EIA-7343-30_AVX-N, symbol Device:CP
- C24: value 330uF -> 100uF/16V; footprint Capacitor_SMD:CP_Elec_8x10 -> Capacitor_Tantalum_SMD:CP_EIA-7343-30_AVX-N
- M1: footprint Connector_JST:JST_PH_S4B-PH-K_1x04_P2.00mm_Horizontal -> TCY_connectors:Amphenol_10114830-11103LF_1x04_P1.25mm_Horizontal; symbol Motor:Stepper_Motor_bipolar -> Connector_Generic_MountingPin:Conn_01x04_MountingPin
Connections:
- net +12V: now also C28.1
- net GND: now also M1.MP (MountPin), C27.2, C28.2
- net REF: now also C27.1
- net at M1.1 (Pin_1): now also U9.7 (OUTA1); no longer U9.8 (OUTA2)
- net at M1.2 (Pin_2): now also U9.8 (OUTA2); no longer U9.7 (OUTA1)
- net at M1.3 (Pin_3): now also U9.11 (OUTB2); no longer U9.12 (OUTB1)
- net at M1.4 (Pin_4): now also U9.12 (OUTB1); no longer U9.11 (OUTB2)
